File: KiCAD/AddressDecoder.kicad_sch (KiCad schematic)
At the start: 11 parts

Commit message: Update schematics (correct page flow) and add alternative to Q4 in BOM
Parts:
- Z3: footprint RetroStackLibrary:TRS80_Model_I_DIP16 -> Package_DIP:DIP-16_W7.62mm; symbol RetroStackLibrary:TRS80ModelIX3 -> RetroStackLibrary:TRS80_Model_I_X3
Changed lines of the file:
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@@
     )
   )
-  (symbol (lib_id "RetroStackLibrary:TRS80ModelIX3") (at 161.925 62.865 0) (unit 1)
+  (symbol (lib_id "RetroStackLibrary:TRS80_Model_I_X3") (at 161.925 62.865 0) (unit 1)
     (in_bom yes) (on_board yes) (dnp no)
     (property "Reference" "Z3" (at 161.925 74.295 0)
@@
       (effects (font (size 1.27 1.27)))
     )
-    (property "Footprint" "RetroStackLibrary:TRS80_Model_I_DIP16" (at 161.925 62.865 0)
+    (property "Footprint" "Package_DIP:DIP-16_W7.62mm" (at 161.925 62.865 0)
       (effects (font (size 1.27 1.27)) hide)
     )

Commit message: Updated revision to Rev C
Other:
- title: TRS-80 Model I G -> TRS-80 Model I Rev G
