File: KiCAD/CPUGating.kicad_sch (KiCad schematic)
At the start: 10 parts

Commit message: Updated revision to Rev C
Parts:
- gave numbers to parts that had none: 2
Other:
- title: TRS-80 Model I G -> TRS-80 Model I Rev G
