File: KiCAD/Keyboard.kicad_sch (KiCad schematic)
At the start: 1 part, among them J100 Connection Mainboard Side

Commit message: Updated revision to Rev C
Other:
- title: TRS-80 Model I G -> TRS-80 Model I Rev G
