File: KiCAD/RAM_ROM_Interface.kicad_sch (KiCad schematic)
At the start: 2 parts

Commit message: Updated revision to Rev C
Connections:
- net D2 is gone; now on net ~{MEM}: Z68.5
- net D6 is gone; now on net ~{MEM}: Z67.5
Other:
- company: (none) -> RetroStack - Marcel Erz
- title: (none) -> TRS-80 Model I Rev G
- moved on the sheet: Z67A, Z67B, Z67C, Z67D, Z68A, Z68B, Z68C, Z68D
