File: KiCAD/RAM_ROM_Interface.kicad_sch (KiCad schematic)
At the start: 2 parts

Commit message: Update to V9
Connections:
- net ~{MEM}: no longer Z67.5, Z68.5
- new net D2: Z68.5
- new net D6: Z67.5
Changed lines of the file:
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@@
 (kicad_sch
-	(version 20231120)
+	(version 20250114)
 	(generator "eeschema")
-	(generator_version "8.0")
+	(generator_version "9.0")
 	(paper "USLetter")
 	(title_block
@@
 	)
 	(junction
-		(at 224.155 100.33)
-		(diameter 0)
-		(color 0 0 0 0)
-	)
-	(junction
 		(at 147.32 87.63)
-		(diameter 0)
-		(color 0 0 0 0)
-	)
-	(junction
-		(at 137.795 74.93)
 		(diameter 0)
 		(color 0 0 0 0)
@@
 	(wire
 		(pts
-			(xy 224.155 100.33) (xy 262.255 100.33)
+			(xy 210.185 100.33) (xy 262.255 100.33)
 		)
 		(stroke
@@
 	(wire
 		(pts
-			(xy 137.795 74.93) (xy 262.255 74.93)
+			(xy 123.825 74.93) (xy 262.255 74.93)
 		)
 		(stroke
@@
 	(wire
 		(pts
-			(xy 210.185 100.33) (xy 224.155 100.33)
-		)
-		(stroke
-			(width 0)
-			(type default)
-		)
-	)
-	(wire
-		(pts
 			(xy 167.005 87.63) (xy 262.255 87.63)
 		)
@@
 		(pts
 			(xy 102.235 68.58) (xy 262.255 68.58)
-		)
-		(stroke
-			(width 0)
-			(type default)
-		)
-	)
-	(wire
-		(pts
-			(xy 123.825 74.93) (xy 137.795 74.93)
 		)
 		(stroke
@@
 	(label "D0"
 		(at 261.62 113.03 180)
-		(fields_autoplaced yes)
 		(effects
 			(font
@@
 	(label "ROMD4"
 		(at 33.655 87.63 0)
-		(fields_autoplaced yes)
 		(effects
 			(font
@@
 	(label "ROMD0"
 		(at 33.655 113.03 0)
-		(fields_autoplaced yes)
 		(effects
 			(font
@@
 	(label "D2"
 		(at 261.62 100.33 180)
-		(fields_autoplaced yes)
 		(effects
 			(font
@@
 	(label "RAMD4"
 		(at 147.32 124.46 270)
-		(fields_autoplaced yes)
 		(effects
 			(font
@@
 	(label "D7"
 		(at 261.62 68.58 180)
-		(fields_autoplaced yes)
 		(effects
 			(font
@@
 	(label "RAMD3"
 		(at 168.91 124.46 270)
-		(fields_autoplaced yes)
 		(effects
 			(font
@@
 	(label "D3"
 		(at 261.62 93.98 180)
-		(fields_autoplaced yes)
 		(effects
 			(font
@@
 	(label "ROMD6"
 		(at 33.655 74.93 0)
-		(fields_autoplaced yes)
 		(effects
 			(font
@@
 	(label "RAMD2"
 		(at 190.5 124.46 270)
-		(fields_autoplaced yes)
 		(effects
 			(font
@@
 	(label "ROMD7"
 		(at 33.655 68.58 0)
-		(fields_autoplaced yes)
 		(effects
 			(font
@@
 	(label "RAMD0"
 		(at 233.68 124.46 270)
-		(fields_autoplaced yes)
 		(effects
 			(font
@@
 	(label "RAMD1"
 		(at 212.09 124.46 270)
-		(fields_autoplaced yes)
 		(effects
 			(font
@@
 	(label "D6"
 		(at 261.62 74.93 180)
-		(fields_autoplaced yes)
 		(effects
 			(font
@@
 	(label "D1"
 		(at 261.62 106.68 180)
-		(fields_autoplaced yes)
 		(effects
 			(font
@@
 	(label "ROMD2"
 		(at 33.655 100.33 0)
-		(fields_autoplaced yes)
 		(effects
 			(font
@@
 	(label "D4"
 		(at 261.62 87.63 180)
-		(fields_autoplaced yes)
 		(effects
 			(font
@@
 	(label "ROMD5"
 		(at 33.655 81.28 0)
-		(fields_autoplaced yes)
 		(effects
 			(font
@@
 	(label "ROMD1"
 		(at 33.655 106.68 0)
-		(fields_autoplaced yes)
 		(effects
 			(font
@@
 	(label "RAMD6"
 		(at 104.14 124.46 270)
-		(fields_autoplaced yes)
 		(effects
 			(font
@@
 	(label "RAMD5"
 		(at 125.73 124.46 270)
-		(fields_autoplaced yes)
 		(effects
 			(font
@@
 	(label "ROMD3"
 		(at 33.655 93.98 0)
-		(fields_autoplaced yes)
 		(effects
 			(font
@@
 	(label "RAMD7"
 		(at 82.55 124.46 270)
-		(fields_autoplaced yes)
 		(effects
 			(font
@@
 	(label "D5"
 		(at 261.62 81.28 180)
-		(fields_autoplaced yes)
 		(effects
 			(font
@@
 		(shape bidirectional)
 		(at 264.795 63.5 90)
-		(fields_autoplaced yes)
 		(effects
 			(font
@@
 		(shape bidirectional)
 		(at 27.305 134.62 180)
-		(fields_autoplaced yes)
 		(effects
 			(font
@@
 		(shape bidirectional)
 		(at 27.305 66.04 180)
-		(fields_autoplaced yes)
 		(effects
 			(font
@@
 		(shape input)
 		(at 27.305 42.545 180)
-		(fields_autoplaced yes)
-		(effects
-			(font
+		(effects
+			(font
