File: KiCAD/ROM.kicad_sch (KiCad schematic)
At the start: 2 parts

Commit message: Update schematics (correct page flow) and add alternative to Q4 in BOM
Parts:
- Z33: footprint RetroStackLibrary:TRS80_Model_I_DIP24 -> Package_DIP:DIP-24_W15.24mm; symbol RetroStackLibrary:2364_20L -> RetroStackLibrary:ROM_2364_20L
- Z34: footprint RetroStackLibrary:TRS80_Model_I_DIP24 -> Package_DIP:DIP-24_W15.24mm; symbol RetroStackLibrary:2332_20L_21L -> RetroStackLibrary:ROM_2332_20L_21L
Changed lines of the file:
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@@
     (effects (font (size 1.27 1.27)) (justify right))
   )
-  (hierarchical_label "ROMD[0..7]" (shape tri_state) (at 128.27 53.34 0) (fields_autoplaced)
+  (hierarchical_label "ROMD[0..7]" (shape bidirectional) (at 128.27 53.34 0) (fields_autoplaced)
     (effects (font (size 1.27 1.27)) (justify left))
   )
@@
     )
   )
-  (symbol (lib_id "RetroStackLibrary:2332_20L_21L") (at 81.915 98.425 0) (unit 1)
+  (symbol (lib_id "RetroStackLibrary:ROM_2332_20L_21L") (at 81.915 98.425 0) (unit 1)
     (in_bom yes) (on_board yes) (dnp no)
     (property "Reference" "Z34" (at 84.455 111.76 0)
@@
       (effects (font (size 1.27 1.27)) (justify left))
     )
-    (property "Footprint" "RetroStackLibrary:TRS80_Model_I_DIP24" (at 81.915 98.425 0)
+    (property "Footprint" "Package_DIP:DIP-24_W15.24mm" (at 81.915 98.425 0)
       (effects (font (size 1.27 1.27)) hide)
     )
@@
     )
   )
-  (symbol (lib_id "RetroStackLibrary:2364_20L") (at 81.915 40.005 0) (unit 1)
+  (symbol (lib_id "RetroStackLibrary:ROM_2364_20L") (at 81.915 40.005 0) (unit 1)
     (in_bom yes) (on_board yes) (dnp no)
     (property "Reference" "Z33" (at 84.455 53.34 0)
@@
       (effects (font (size 1.27 1.27)) (justify left))
     )
-    (property "Footprint" "RetroStackLibrary:TRS80_Model_I_DIP24" (at 81.915 40.005 0)
+    (property "Footprint" "Package_DIP:DIP-24_W15.24mm" (at 81.915 40.005 0)
       (effects (font (size 1.27 1.27)) hide)
     )

Commit message: Updated revision to Rev C
Other:
- title: TRS-80 Model I G -> TRS-80 Model I Rev G
