File: KiCAD/TRS80_Model_I_G_E1.kicad_pcb (KiCad board)
At the start: 2 copper layers, 407 x 184 mm, 231 parts, among them J1 Front View, J100 Connection Mainboard Side, J2 Front View, J3 Front View, J4 Edge Connector, K1 Relay_SPST-NO, Q1 2N3904, Q2 2N3906, Q3 TIP29A, Q4 2N6594, Q5 2N3906, Q6 MJE34, Y1 10.6445 MHz

Commit message: New labels file and updated BOM
Parts:
- C1: value 220uF 16V -> 220uF
- C10, C11, C2, C4, C5, C57: value 10uF 16V -> 10uF
- C14, C15: value 0.01uF 25V -> 0.01uF
- C16, C17, C18, C19, C22, C23, C29, C31, C33, C35, C36, C37, C38, C40, C41, C44, C45, C46, C47, C48, C49, C50, C51, C52, C53, C54, C55, C56, C58, C_C58: value 0.1uF 12V -> 0.1uF
- C42: value 22uF 16V -> 22uF
- C6: value 100uF 16V -> 100uF
- CR1: value 1N4735 -> 4735
- CR10, CR9: value 1N982 -> 982
- CR2: value 1N5231 -> 5231
- CR3, CR4, CR5, CR6, CR7: value 1N4148 -> 4148
- CR8: value MDA202 -> MDA202 (KBP210)
- C_R67: value 100 -> 220
- J1: value Front View -> Power Connector
- J2: value Front View -> Video Connector
- J3: value Front View -> Cassette Connector
- K1: value Relay_SPST-NO -> Relay
- Q4: value 2N6594 -> 2N6594 (RS2040)
- Q6: value MJE34 -> MJE34 (TIP32C)
- S1: value ~ -> Power
- Z13, Z14, Z15, Z16, Z17, Z19, Z20: value MK4116 -> 4116
- Z18: value MK4116 -> 41116
- Z3, Z71: value ~ -> Mem Config
- Z33: value 2364_20L -> 2364 (ROM A)
- Z34: value 2332_20L_21L -> 2332 (ROM B)
- Z40: value Z80CPU -> Z80 CPU

Commit message: Updated revision to Rev C
Parts:
- removed REF**: OSHW-Symbol_6.7x6mm_Copper, Symbol:OSHW-Symbol_6.7x6mm_Copper
- C1: value 220uF -> 220uF 16V
- C10, C11, C2, C4, C5, C57: value 10uF -> 10uF 16V
- C14, C15, C3, C7: value 0.01uF -> 0.01uF 24V
- C16, C17, C18, C19, C22, C23, C29, C31, C33, C35, C36, C37, C38, C39, C40, C41, C44, C45, C46, C47, C48, C49, C50, C51, C52, C53, C54, C55, C56, C58, C_C58: value 0.1uF -> 0.1uF 12V
- C28, C30, C32, C34: value 0.1uF -> 0.1uF 25V
- C42: value 22uF -> 22uF 16V
- C6: value 100uF -> 100uF 16V
- CR1: value 4735 -> 1N4735
- CR10, CR9: value 982 -> 1N982
- CR2: value 5231 -> 1N5231
- CR3, CR4, CR5, CR6, CR7: value 4148 -> 1N4148
- CR8: value MDA202 (KBP210) -> MDA202
- J1: value Power Connector -> Front View
- J2: value Video Connector -> Front View
- J3: value Cassette Connector -> Front View
- K1: value Relay -> Relay_SPST-NO
- Q4: value 2N6594 (RS2040) -> 2N6594
- Q6: value MJE34 (TIP32C) -> MJE34
- S1: value Power -> ~
- Z18: value 41116 -> 4116
- Z3, Z71: value Mem Config -> ~
- Z33: value 2364 (ROM A) -> 2364_20L
- Z34: value 2332 (ROM B) -> 2332_20L_21L
- Z40: value Z80 CPU -> Z80CPU
- moved Z33 0.41 mm to (178.6, 159.0)
Connections:
- net /RAM/ROMD0 renamed /RAM-ROM Interface/ROMD0
- net /RAM/ROMD1 renamed /RAM-ROM Interface/ROMD1
- net /RAM/ROMD2 renamed /RAM-ROM Interface/ROMD2
- net /RAM/ROMD3 renamed /RAM-ROM Interface/ROMD3
- net /RAM/ROMD4 renamed /RAM-ROM Interface/ROMD4
- net /RAM/ROMD5 renamed /RAM-ROM Interface/ROMD5
- net /RAM/ROMD6 renamed /RAM-ROM Interface/ROMD6
- net /RAM/ROMD7 renamed /RAM-ROM Interface/ROMD7
Routing:
- net GND: track 4094.7 -> 4209.2 mm
- net Net-(Q6-C): track 73.2 -> 56.0 mm
- net /A6: track 611.6 -> 610.9 mm
- net /A7: track 514.0 -> 513.4 mm
Other:
- board text added: "E1C"
- board text added: "Replicated By: RetroStack Marcel Erz"
- board text removed: "Created By: Marcel Erz"
- board text removed: "E1B"
