File: KiCAD/Video Latch.kicad_sch (KiCad schematic)
At the start: 6 parts

Commit message: Update to V9
Changed lines of the file:
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@@
 (kicad_sch
-	(version 20231120)
+	(version 20250114)
 	(generator "eeschema")
-	(generator_version "8.0")
+	(generator_version "9.0")
 	(paper "USLetter")
 	(title_block
@@
 		(comment 4 "Video Latch")
 	)
+	(text "CHARGAP"
+		(exclude_from_sim no)
+		(at 133.35 49.53 0)
+		(effects
+			(font
+				(size 1 1)
+			)
+			(justify left bottom)
+		)
+	)
+	(text "GRAPHICS"
+		(exclude_from_sim no)
+		(at 100.33 34.925 0)
+		(effects
+			(font
+				(size 1 1)
+			)
+			(justify left bottom)
+		)
+	)
+	(text "Clear when CPU drives"
+		(exclude_from_sim no)
+		(at 125.73 86.995 0)
+		(effects
+			(font
+				(size 1 1)
+			)
+			(justify left bottom)
+		)
+	)
+	(text "~{BLANK}"
+		(exclude_from_sim no)
+		(at 123.19 44.45 0)
+		(effects
+			(font
+				(size 1 1)
+			)
+			(justify left bottom)
+		)
+	)
+	(text "~{GRAPHICS}"
+		(exclude_from_sim no)
+		(at 133.35 34.925 0)
+		(effects
+			(font
+				(size 1 1)
+			)
+			(justify left bottom)
+		)
+	)
 	(junction
 		(at 107.95 113.665)
@@
 		)
 	)
-	(text "CHARGAP"
-		(exclude_from_sim no)
-		(at 133.35 49.53 0)
-		(effects
-			(font
-				(size 1 1)
-			)
-			(justify left bottom)
-		)
-	)
-	(text "GRAPHICS"
-		(exclude_from_sim no)
-		(at 100.33 34.925 0)
-		(effects
-			(font
-				(size 1 1)
-			)
-			(justify left bottom)
-		)
-	)
-	(text "Clear when CPU drives"
-		(exclude_from_sim no)
-		(at 125.73 86.995 0)
-		(effects
-			(font
-				(size 1 1)
-			)
-			(justify left bottom)
-		)
-	)
-	(text "~{BLANK}"
-		(exclude_from_sim no)
-		(at 123.19 44.45 0)
-		(effects
-			(font
-				(size 1 1)
-			)
-			(justify left bottom)
-		)
-	)
-	(text "~{GRAPHICS}"
-		(exclude_from_sim no)
-		(at 133.35 34.925 0)
-		(effects
-			(font
-				(size 1 1)
-			)
-			(justify left bottom)
-		)
-	)
 	(label "LB0"
 		(at 189.865 128.905 0)
-		(fields_autoplaced yes)
 		(effects
 			(font
@@
 	(label "VD4"
 		(at 95.25 118.745 180)
-		(fields_autoplaced yes)
 		(effects
 			(font
@@
 	(label "VD1"
 		(at 95.25 126.365 180)
-		(fields_autoplaced yes)
 		(effects
 			(font
@@
 	(label "~{VCLR}"
 		(at 130.175 85.09 0)
-		(fields_autoplaced yes)
 		(effects
 			(font
@@
 	(label "VD0"
 		(at 95.25 128.905 180)
-		(fields_autoplaced yes)
 		(effects
 			(font
@@
 	(label "LB4"
 		(at 189.865 118.745 0)
-		(fields_autoplaced yes)
 		(effects
 			(font
@@
 	(label "VD5"
 		(at 95.25 123.825 180)
-		(fields_autoplaced yes)
 		(effects
 			(font
@@
 	(label "LB3"
 		(at 189.865 121.285 0)
-		(fields_autoplaced yes)
 		(effects
 			(font
@@
 	(label "LB6"
 		(at 189.865 54.61 0)
-		(fields_autoplaced yes)
 		(effects
 			(font
@@
 	(label "LB5"
 		(at 189.865 123.825 0)
-		(fields_autoplaced yes)
 		(effects
 			(font
@@
 	(label "LB1"
 		(at 189.865 126.365 0)
-		(fields_autoplaced yes)
 		(effects
 			(font
@@
 	(label "VD2"
 		(at 95.25 116.205 180)
-		(fields_autoplaced yes)
 		(effects
 			(font
@@
 	(label "VD3"
 		(at 95.25 121.285 180)
-		(fields_autoplaced yes)
 		(effects
 			(font
@@
 	(label "VD7"
 		(at 95.25 34.925 180)
-		(fields_autoplaced yes)
 		(effects
 			(font
@@
 	(label "VD6"
 		(at 95.25 54.61 180)
-		(fields_autoplaced yes)
 		(effects
 			(font
@@
 	(label "LB2"
 		(at 189.865 116.205 0)
-		(fields_autoplaced yes)
 		(effects
 			(font
@@
 		(shape input)
 		(at 127 49.53 180)
-		(fields_autoplaced yes)
 		(effects
 			(font
@@
 		(shape output)
 		(at 213.36 50.8 0)
-		(fields_autoplaced yes)
 		(effects
 			(font
@@
 		(shape output)
 		(at 175.895 44.45 0)
-		(fields_autoplaced yes)
 		(effects
 			(font
@@
 		(shape input)
 		(at 118.11 74.93 90)
-		(fields_autoplaced yes)
 		(effects
 			(font
@@
 		(shape output)
 		(at 175.895 39.37 0)
-		(fields_autoplaced yes)
 		(effects
 			(font
@@
 		(shape input)
 		(at 104.14 133.985 180)
-		(fields_autoplaced yes)
 		(effects
 			(font
@@
 		(shape output)
 		(at 175.895 41.91 0)
-		(fields_autoplaced yes)
 		(effects
 			(font
@@
 		(shape input)
 		(at 104.775 46.99 180)
-		(fields_autoplaced yes)
 		(effects
 			(font
@@
 		(shape input)
 		(at 71.755 31.115 180)
-		(fields_autoplaced yes)
 		(effects
 			(font
@@
 		(shape input)
 		(at 104.775 41.91 180)
-		(fields_autoplaced yes)
 		(effects
 			(font
@@
 		(shape output)
 		(at 175.895 52.07 0)
-		(fields_autoplaced yes)
-		(effects
-			(font
+		(effects
+			(font
