File: KiCAD/VideoGen.kicad_sch (KiCad schematic)
At the start: 13 parts

Commit message: Update schematics (correct page flow) and add alternative to Q4 in BOM
Parts:
- Z29: footprint RetroStackLibrary:TRS80_Model_I_DIP18 -> Package_DIP:DIP-18_W7.62mm
Changed lines of the file:
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@@
       (effects (font (size 1 1)))
     )
-    (property "Footprint" "RetroStackLibrary:TRS80_Model_I_DIP18" (at 78.74 31.115 0)
+    (property "Footprint" "Package_DIP:DIP-18_W7.62mm" (at 78.74 31.115 0)
       (effects (font (size 1.27 1.27)) hide)
     )

Commit message: Updated revision to Rev C
Parts:
- gave numbers to parts that had none: 1
Other:
- note added: "Character Generators: - Motorola 3108001 (floating "a") - Motorola MCM6670 (fixed floating "a") - Motorola 8046673 SCM37530 (latest)"
- title: TRS-80 Model I G -> TRS-80 Model I Rev G
