File: KiCAD/VideoGen.kicad_sch (KiCad schematic)
At the start: 9 parts

Commit message: Update to V9
Parts:
- renumbered Z42 to Z9
Changed lines of the file:
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@@
 (kicad_sch
-	(version 20231120)
+	(version 20250114)
 	(generator "eeschema")
-	(generator_version "8.0")
+	(generator_version "9.0")
 	(paper "USLetter")
 	(title_block
@@
 		(comment 4 "Video Generator")
 	)
+	(text "ASCII"
+		(exclude_from_sim no)
+		(at 88.265 91.44 0)
+		(effects
+			(font
+				(size 1.27 1.27)
+			)
+			(justify left bottom)
+		)
+	)
+	(text "Character Generators:\n- Motorola 3108001 (floating \"a\")\n- Motorola MCM6670 (fixed floating \"a\")\n- Motorola 8046673 SCM37530 (latest)"
+		(exclude_from_sim no)
+		(at 217.805 26.67 0)
+		(effects
+			(font
+				(size 1.27 1.27)
+			)
+			(justify left bottom)
+		)
+	)
+	(text "SHIFT/~{LOAD}"
+		(exclude_from_sim no)
+		(at 88.265 113.665 0)
+		(effects
+			(font
+				(size 1.27 1.27)
+			)
+			(justify left bottom)
+		)
+	)
+	(text "LATCH"
+		(exclude_from_sim no)
+		(at 69.85 99.695 0)
+		(effects
+			(font
+				(size 1 1)
+			)
+			(justify right bottom)
+		)
+	)
+	(text "Right"
+		(exclude_from_sim no)
+		(at 97.155 133.985 0)
+		(effects
+			(font
+				(size 1.27 1.27)
+			)
+			(justify left bottom)
+		)
+	)
+	(text "GRAPHICS\nPIXEL"
+		(exclude_from_sim no)
+		(at 163.195 121.285 0)
+		(effects
+			(font
+				(size 1.27 1.27)
+			)
+			(justify left bottom)
+		)
+	)
+	(text "Left"
+		(exclude_from_sim no)
+		(at 97.155 138.43 0)
+		(effects
+			(font
+				(size 1.27 1.27)
+			)
+			(justify left bottom)
+		)
+	)
+	(text "LATCH"
+		(exclude_from_sim no)
+		(at 69.85 119.38 0)
+		(effects
+			(font
+				(size 1 1)
+			)
+			(justify right bottom)
+		)
+	)
+	(text "SHIFT/~{LOAD}"
+		(exclude_from_sim no)
+		(at 88.265 93.98 0)
+		(effects
+			(font
+				(size 1.27 1.27)
+			)
+			(justify left bottom)
+		)
+	)
+	(text "Character Generator"
+		(exclude_from_sim no)
+		(at 76.835 60.325 90)
+		(effects
+			(font
+				(size 1 1)
+			)
+			(justify left bottom)
+		)
+	)
+	(text "GRAPHICS"
+		(exclude_from_sim no)
+		(at 88.265 111.125 0)
+		(effects
+			(font
+				(size 1.27 1.27)
+			)
+			(justify left bottom)
+		)
+	)
+	(text "~{SHIFT}"
+		(exclude_from_sim no)
+		(at 102.235 21.59 0)
+		(effects
+			(font
+				(size 1.27 1.27)
+			)
+			(justify left bottom)
+		)
+	)
+	(text "ASCII\nPIXEL"
+		(exclude_from_sim no)
+		(at 163.195 31.75 0)
+		(effects
+			(font
+				(size 1.27 1.27)
+			)
+			(justify left bottom)
+		)
+	)
+	(text "Inversed Clock\n(delays clock)"
+		(exclude_from_sim no)
+		(at 72.39 16.51 0)
+		(effects
+			(font
+				(size 1 1)
+			)
+			(justify left bottom)
+		)
+	)
 	(junction
 		(at 57.785 90.17)
@@
 		)
 	)
-	(text "ASCII"
-		(exclude_from_sim no)
-		(at 88.265 91.44 0)
-		(effects
-			(font
-				(size 1.27 1.27)
-			)
-			(justify left bottom)
-		)
-	)
-	(text "Character Generators:\n- Motorola 3108001 (floating \"a\")\n- Motorola MCM6670 (fixed floating \"a\")\n- Motorola 8046673 SCM37530 (latest)"
-		(exclude_from_sim no)
-		(at 217.805 26.67 0)
-		(effects
-			(font
-				(size 1.27 1.27)
-			)
-			(justify left bottom)
-		)
-	)
-	(text "SHIFT/~{LOAD}"
-		(exclude_from_sim no)
-		(at 88.265 113.665 0)
-		(effects
-			(font
-				(size 1.27 1.27)
-			)
-			(justify left bottom)
-		)
-	)
-	(text "LATCH"
-		(exclude_from_sim no)
-		(at 69.85 99.695 0)
-		(effects
-			(font
-				(size 1 1)
-			)
-			(justify right bottom)
-		)
-	)
-	(text "Right"
-		(exclude_from_sim no)
-		(at 97.155 133.985 0)
-		(effects
-			(font
-				(size 1.27 1.27)
-			)
-			(justify left bottom)
-		)
-	)
-	(text "GRAPHICS\nPIXEL"
-		(exclude_from_sim no)
-		(at 163.195 121.285 0)
-		(effects
-			(font
-				(size 1.27 1.27)
-			)
-			(justify left bottom)
-		)
-	)
-	(text "Left"
-		(exclude_from_sim no)
-		(at 97.155 138.43 0)
-		(effects
-			(font
-				(size 1.27 1.27)
-			)
-			(justify left bottom)
-		)
-	)
-	(text "LATCH"
-		(exclude_from_sim no)
-		(at 69.85 119.38 0)
-		(effects
-			(font
-				(size 1 1)
-			)
-			(justify right bottom)
-		)
-	)
-	(text "SHIFT/~{LOAD}"
-		(exclude_from_sim no)
-		(at 88.265 93.98 0)
-		(effects
-			(font
-				(size 1.27 1.27)
-			)
-			(justify left bottom)
-		)
-	)
-	(text "Character Generator"
-		(exclude_from_sim no)
-		(at 76.835 60.325 90)
-		(effects
-			(font
-				(size 1 1)
-			)
-			(justify left bottom)
-		)
-	)
-	(text "GRAPHICS"
-		(exclude_from_sim no)
-		(at 88.265 111.125 0)
-		(effects
-			(font
-				(size 1.27 1.27)
-			)
-			(justify left bottom)
-		)
-	)
-	(text "~{SHIFT}"
-		(exclude_from_sim no)
-		(at 102.235 21.59 0)
-		(effects
-			(font
-				(size 1.27 1.27)
-			)
-			(justify left bottom)
-		)
-	)
-	(text "ASCII\nPIXEL"
-		(exclude_from_sim no)
-		(at 163.195 31.75 0)
-		(effects
-			(font
-				(size 1.27 1.27)
-			)
-			(justify left bottom)
-		)
-	)
-	(text "Inversed Clock\n(delays clock)"
-		(exclude_from_sim no)
-		(at 72.39 16.51 0)
-		(effects
-			(font
-				(size 1 1)
-			)
-			(justify left bottom)
-		)
-	)
 	(label "LB3"
 		(at 55.245 156.845 0)
-		(fields_autoplaced yes)
 		(effects
 			(font
@@
 	(label "LB2"
 		(at 55.245 139.065 0)
-		(fields_autoplaced yes)
 		(effects
 			(font
@@
 	(label "LB6"
 		(at 55.245 54.61 0)
-		(fields_autoplaced yes)
 		(effects
 			(font
@@
 	(label "LB0"
 		(at 55.245 39.37 0)
-		(fields_autoplaced yes)
 		(effects
 			(font
@@
 	(label "LB0"
 		(at 55.245 136.525 0)
-		(fields_autoplaced yes)
 		(effects
 			(font
@@
 	(label "LB4"
 		(at 55.245 141.605 0)
-		(fields_autoplaced yes)
 		(effects
 			(font
@@
 	(label "LB4"
 		(at 55.245 49.53 0)
-		(fields_autoplaced yes)
 		(effects
 			(font
@@
 	(label "L2"
 		(at 55.245 64.77 0)
-		(fields_autoplaced yes)
 		(effects
 			(font
@@
 	(label "LB1"
 		(at 55.245 154.305 0)
-		(fields_autoplaced yes)
 		(effects
 			(font
@@
 	(label "L1"
 		(at 55.245 62.23 0)
-		(fields_autoplaced yes)
 		(effects
 			(font
@@
 	(label "LB3"
 		(at 55.245 46.99 0)
-		(fields_autoplaced yes)
 		(effects
 			(font
@@
 	(label "L2"
 		(at 55.245 172.085 0)
-		(fields_autoplaced yes)
 		(effects
 			(font
@@
 	(label "L3"
 		(at 55.245 174.625 0)
-		(fields_autoplaced yes)
 		(effects
 			(font
@@
 	(label "LB2"
 		(at 55.245 44.45 0)
-		(fields_autoplaced yes)
 		(effects
 			(font
@@
 	(label "LB5"
 		(at 55.245 159.385 0)
-		(fields_autoplaced yes)
 		(effects
 			(font
@@
 	(label "LB1"
 		(at 55.245 41.91 0)
-		(fields_autoplaced yes)
 		(effects
 			(font
@@
 	(label "L0"
 		(at 55.245 59.69 0)
-		(fields_autoplaced yes)
 		(effects
 			(font
@@
 	(label "LB5"
 		(at 55.245 52.07 0)
-		(fields_autoplaced yes)
 		(effects
 			(font
@@
 		(shape input)
 		(at 27.94 35.56 180)
-		(fields_autoplaced yes)
 		(effects
 			(font
@@
 		(shape input)
 		(at 27.94 90.17 180)
-		(fields_autoplaced yes)
 		(effects
 			(font
@@
 		(shape input)
 		(at 71.12 114.935 180)
-		(fields_autoplaced yes)
 		(effects
 			(font
@@
 		(shape input)
 		(at 27.94 163.195 180)
-		(fields_autoplaced yes)
 		(effects
 			(font
@@
 		(shape input)
 		(at 71.12 95.25 180)
-		(fields_autoplaced yes)
 		(effects
 			(font
@@
 		(shape input)
 		(at 32.385 21.59 180)
-		(fields_autoplaced yes)
 		(effects
 			(font
@@
 		(shape input)
 		(at 71.12 92.71 180)
-		(fields_autoplaced yes)
 		(effects
 			(font
@@
 		(shape input)
 		(at 27.94 104.14 180)
-		(fields_autoplaced yes)
 		(effects
 			(font
@@
 		(shape output)
 		(at 204.47 91.44 0)
-		(fields_autoplaced yes)
 		(effects
 			(font
@@
 		(on_board yes)
 		(dnp no)
-		(property "Reference" "Z42"
+		(property "Reference" "Z9"
 			(at 80.01 18.415 0)
 			(effects
