File: KiCAD/VideoMixer.kicad_sch (KiCad schematic)
At the start: 12 parts, among them J2 Front View, Q1 2N3904, Q2 2N3906

Commit message: Updated revision to Rev C
Other:
- title: TRS-80 Model I G -> TRS-80 Model I Rev G
