File: KiCAD/VideoRAM.kicad_sch (KiCad schematic)
At the start: 10 parts

Commit message: Update schematics (correct page flow) and add alternative to Q4 in BOM
Parts:
- Z45, Z46, Z47, Z48, Z61, Z62, Z63: footprint RetroStackLibrary:TRS80_Model_I_DIP16 -> Package_DIP:DIP-16_W7.62mm; symbol RetroStackLibrary:2102 -> RetroStackLibrary:SRAM_2102
Changed lines of the file:
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@@
     )
   )
-  (symbol (lib_id "RetroStackLibrary:2102") (at 210.82 78.74 0) (unit 1)
+  (symbol (lib_id "RetroStackLibrary:SRAM_2102") (at 210.82 78.74 0) (unit 1)
     (in_bom yes) (on_board yes) (dnp no)
     (property "Reference" "Z48" (at 203.2 81.915 0)
@@
       (effects (font (size 1 1)))
     )
-    (property "Footprint" "RetroStackLibrary:TRS80_Model_I_DIP16" (at 210.82 78.74 0)
+    (property "Footprint" "Package_DIP:DIP-16_W7.62mm" (at 210.82 78.74 0)
       (effects (font (size 1.27 1.27)) hide)
     )
@@
     )
   )
-  (symbol (lib_name "2102_1") (lib_id "RetroStackLibrary:2102") (at 78.105 78.74 0) (unit 1)
+  (symbol (lib_id "RetroStackLibrary:SRAM_2102") (at 78.105 78.74 0) (unit 1)
     (in_bom yes) (on_board yes) (dnp no)
     (property "Reference" "Z63" (at 70.485 81.915 0)
@@
       (effects (font (size 1 1)))
     )
-    (property "Footprint" "RetroStackLibrary:TRS80_Model_I_DIP16" (at 78.105 78.74 0)
+    (property "Footprint" "Package_DIP:DIP-16_W7.62mm" (at 78.105 78.74 0)
       (effects (font (size 1.27 1.27)) hide)
     )
@@
     )
   )
-  (symbol (lib_name "2102_3") (lib_id "RetroStackLibrary:2102") (at 121.92 78.74 0) (unit 1)
+  (symbol (lib_id "RetroStackLibrary:SRAM_2102") (at 121.92 78.74 0) (unit 1)
     (in_bom yes) (on_board yes) (dnp no)
     (property "Reference" "Z61" (at 114.3 81.915 0)
@@
       (effects (font (size 1 1)))
     )
-    (property "Footprint" "RetroStackLibrary:TRS80_Model_I_DIP16" (at 121.92 78.74 0)
+    (property "Footprint" "Package_DIP:DIP-16_W7.62mm" (at 121.92 78.74 0)
       (effects (font (size 1.27 1.27)) hide)
     )
@@
     )
   )
-  (symbol (lib_name "2102_2") (lib_id "RetroStackLibrary:2102") (at 99.695 78.74 0) (unit 1)
+  (symbol (lib_id "RetroStackLibrary:SRAM_2102") (at 99.695 78.74 0) (unit 1)
     (in_bom yes) (on_board yes) (dnp no)
     (property "Reference" "Z62" (at 92.075 81.915 0)
@@
       (effects (font (size 1 1)))
     )
-    (property "Footprint" "RetroStackLibrary:TRS80_Model_I_DIP16" (at 99.695 78.74 0)
+    (property "Footprint" "Package_DIP:DIP-16_W7.62mm" (at 99.695 78.74 0)
       (effects (font (size 1.27 1.27)) hide)
     )
@@
     )
   )
-  (symbol (lib_name "2102_4") (lib_id "RetroStackLibrary:2102") (at 144.145 78.74 0) (unit 1)
+  (symbol (lib_id "RetroStackLibrary:SRAM_2102") (at 144.145 78.74 0) (unit 1)
     (in_bom yes) (on_board yes) (dnp no)
     (property "Reference" "Z45" (at 136.525 81.915 0)
@@
       (effects (font (size 1 1)))
     )
-    (property "Footprint" "RetroStackLibrary:TRS80_Model_I_DIP16" (at 144.145 78.74 0)
+    (property "Footprint" "Package_DIP:DIP-16_W7.62mm" (at 144.145 78.74 0)
       (effects (font (size 1.27 1.27)) hide)
     )
@@
     )
   )
-  (symbol (lib_name "2102_5") (lib_id "RetroStackLibrary:2102") (at 166.37 78.74 0) (unit 1)
+  (symbol (lib_id "RetroStackLibrary:SRAM_2102") (at 166.37 78.74 0) (unit 1)
     (in_bom yes) (on_board yes) (dnp no)
     (property "Reference" "Z46" (at 158.75 81.915 0)
@@
       (effects (font (size 1 1)))
     )
-    (property "Footprint" "RetroStackLibrary:TRS80_Model_I_DIP16" (at 166.37 78.74 0)
+    (property "Footprint" "Package_DIP:DIP-16_W7.62mm" (at 166.37 78.74 0)
       (effects (font (size 1.27 1.27)) hide)
     )
@@
     )
   )
-  (symbol (lib_name "2102_6") (lib_id "RetroStackLibrary:2102") (at 188.595 78.74 0) (unit 1)
+  (symbol (lib_id "RetroStackLibrary:SRAM_2102") (at 188.595 78.74 0) (unit 1)
     (in_bom yes) (on_board yes) (dnp no)
     (property "Reference" "Z47" (at 180.975 81.915 0)
@@
       (effects (font (size 1 1)))
     )
-    (property "Footprint" "RetroStackLibrary:TRS80_Model_I_DIP16" (at 188.595 78.74 0)
-      (effects (font (size 1.27 1.27)) hide)
-    )
+    (property "Footprint" "Package_DIP:DIP-16_W7.62mm" (at 188.595 78.74 0)
+      (effects (font (size 1.27 1.27)) hide)
+    )

Commit message: Updated revision to Rev C
Other:
- title: TRS-80 Model I G -> TRS-80 Model I Rev G
