File: KiCAD/VideoSync.kicad_sch (KiCad schematic)
At the start: 11 parts

Commit message: Updated revision to Rev C
Other:
- note added: "Amplifier"
- note removed: "Level Shifter"
- title: TRS-80 Model I G -> TRS-80 Model I Rev G
